Commit message: save models pkls log structure better

File: car/husky/husky.urdf (robot description, URDF)
Before this commit: robot husky_robot, 11 links, 10 joints
Links:
- link base_footprint: mass None -> 0.001
- link front_bumper_link: mass None -> 0.1
- link imu_link: mass None -> 0.001
- link rear_bumper_link: mass None -> 0.1
- link top_plate_link: mass None -> 0.1
- link user_rail_link: mass None -> 0.1
